File: pcb/LEDs.sch (KiCad schematic (older format))
At the start: 15 parts, among them Q2 S9013, Q3 S9013, Q4 S9013

Commit message: Cleanup libs
Parts:
- Q2, Q3, Q4: symbol JLC_Parts:S9013 -> LCSC_parts:S9013
Changed lines of the file:
@@
 $EndComp
 $Comp
-L JLC_Parts:S9013 Q?
+L LCSC_parts:S9013 Q?
 U 1 1 60377CC9
 P 3200 4150
@@
 $EndComp
 $Comp
-L JLC_Parts:S9013 Q?
+L LCSC_parts:S9013 Q?
 U 1 1 60383DF4
 P 5300 4150
@@
 $EndComp
 $Comp
-L JLC_Parts:S9013 Q?
+L LCSC_parts:S9013 Q?
 U 1 1 60387BD9
 P 7400 4150

Commit message: Added switches
Parts:
- R23, R26, R29: value 100R -> 200R; footprint Resistor_SMD:R_0603_1608Metric -> Resistor_SMD:R_0603_1608Metric_Pad0.98x0.95mm_HandSolder
- R24, R27, R30: value 100k -> 100K; footprint Resistor_SMD:R_0603_1608Metric -> Resistor_SMD:R_0603_1608Metric_Pad0.98x0.95mm_HandSolder
- R25, R28, R31: value 150R -> 200R; footprint Resistor_SMD:R_0603_1608Metric -> Resistor_SMD:R_0603_1608Metric_Pad0.98x0.95mm_HandSolder
Changed lines of the file:
@@
 $Descr A4 11693 8268
 encoding utf-8
-Sheet 13 13
+Sheet 13 15
 Title ""
 Date ""
@@
 AR Path="/6036720E/60377CD5" Ref="R23"  Part="1"
 F 0 "R23" V 2293 4150 50  0000 C CNN
-F 1 "100R" V 2384 4150 50  0000 C CNN
-F 2 "Resistor_SMD:R_0603_1608Metric" V 2430 4150 50  0001 C CNN
+F 1 "200R" V 2384 4150 50  0000 C CNN
+F 2 "Resistor_SMD:R_0603_1608Metric_Pad0.98x0.95mm_HandSolder" V 2430 4150 50  0001 C CNN
 F 3 "~" H 2500 4150 50  0001 C CNN
 	1    2500 4150
@@
 AR Path="/6036720E/60377CDB" Ref="R24"  Part="1"
 F 0 "R24" H 2780 4354 50  0000 R CNN
-F 1 "100k" H 2780 4445 50  0000 R CNN
-F 2 "Resistor_SMD:R_0603_1608Metric" V 2780 4400 50  0001 C CNN
+F 1 "100K" H 2780 4445 50  0000 R CNN
+F 2 "Resistor_SMD:R_0603_1608Metric_Pad0.98x0.95mm_HandSolder" V 2780 4400 50  0001 C CNN
 F 3 "~" H 2850 4400 50  0001 C CNN
 	1    2850 4400
@@
 AR Path="/6036720E/60383E00" Ref="R26"  Part="1"
 F 0 "R26" V 4393 4150 50  0000 C CNN
-F 1 "100R" V 4484 4150 50  0000 C CNN
-F 2 "Resistor_SMD:R_0603_1608Metric" V 4530 4150 50  0001 C CNN
+F 1 "200R" V 4484 4150 50  0000 C CNN
+F 2 "Resistor_SMD:R_0603_1608Metric_Pad0.98x0.95mm_HandSolder" V 4530 4150 50  0001 C CNN
 F 3 "~" H 4600 4150 50  0001 C CNN
 	1    4600 4150
@@
 AR Path="/6036720E/60383E06" Ref="R27"  Part="1"
 F 0 "R27" H 4880 4354 50  0000 R CNN
-F 1 "100k" H 4880 4445 50  0000 R CNN
-F 2 "Resistor_SMD:R_0603_1608Metric" V 4880 4400 50  0001 C CNN
+F 1 "100K" H 4880 4445 50  0000 R CNN
+F 2 "Resistor_SMD:R_0603_1608Metric_Pad0.98x0.95mm_HandSolder" V 4880 4400 50  0001 C CNN
 F 3 "~" H 4950 4400 50  0001 C CNN
 	1    4950 4400
@@
 AR Path="/6036720E/60387BE5" Ref="R29"  Part="1"
 F 0 "R29" V 6493 4150 50  0000 C CNN
-F 1 "100R" V 6584 4150 50  0000 C CNN
-F 2 "Resistor_SMD:R_0603_1608Metric" V 6630 4150 50  0001 C CNN
+F 1 "200R" V 6584 4150 50  0000 C CNN
+F 2 "Resistor_SMD:R_0603_1608Metric_Pad0.98x0.95mm_HandSolder" V 6630 4150 50  0001 C CNN
 F 3 "~" H 6700 4150 50  0001 C CNN
 	1    6700 4150
@@
 AR Path="/6036720E/60387BEB" Ref="R30"  Part="1"
 F 0 "R30" H 6980 4354 50  0000 R CNN
-F 1 "100k" H 6980 4445 50  0000 R CNN
-F 2 "Resistor_SMD:R_0603_1608Metric" V 6980 4400 50  0001 C CNN
+F 1 "100K" H 6980 4445 50  0000 R CNN
+F 2 "Resistor_SMD:R_0603_1608Metric_Pad0.98x0.95mm_HandSolder" V 6980 4400 50  0001 C CNN
 F 3 "~" H 7050 4400 50  0001 C CNN
 	1    7050 4400
@@
 AR Path="/6036720E/60399B8F" Ref="R25"  Part="1"
 F 0 "R25" H 3230 3204 50  0000 R CNN
-F 1 "150R" H 3230 3295 50  0000 R CNN
-F 2 "Resistor_SMD:R_0603_1608Metric" V 3230 3250 50  0001 C CNN
+F 1 "200R" H 3230 3295 50  0000 R CNN
+F 2 "Resistor_SMD:R_0603_1608Metric_Pad0.98x0.95mm_HandSolder" V 3230 3250 50  0001 C CNN
 F 3 "~" H 3300 3250 50  0001 C CNN
 	1    3300 3250
@@
 AR Path="/6036720E/6039D17A" Ref="R28"  Part="1"
 F 0 "R28" H 5330 3204 50  0000 R CNN
-F 1 "150R" H 5330 3295 50  0000 R CNN
-F 2 "Resistor_SMD:R_0603_1608Metric" V 5330 3250 50  0001 C CNN
+F 1 "200R" H 5330 3295 50  0000 R CNN
+F 2 "Resistor_SMD:R_0603_1608Metric_Pad0.98x0.95mm_HandSolder" V 5330 3250 50  0001 C CNN
 F 3 "~" H 5400 3250 50  0001 C CNN
 	1    5400 3250
@@
 AR Path="/6036720E/6039DCC9" Ref="R31"  Part="1"
 F 0 "R31" H 7430 3204 50  0000 R CNN
-F 1 "150R" H 7430 3295 50  0000 R CNN
-F 2 "Resistor_SMD:R_0603_1608Metric" V 7430 3250 50  0001 C CNN
+F 1 "200R" H 7430 3295 50  0000 R CNN
+F 2 "Resistor_SMD:R_0603_1608Metric_Pad0.98x0.95mm_HandSolder" V 7430 3250 50  0001 C CNN
 F 3 "~" H 7500 3250 50  0001 C CNN
 	1    7500 3250
