File: pcb/USB_serial.sch (KiCad schematic (older format))
At the start: 4 parts, among them J1 USB_B_Micro, U5 CH340K

Commit message: Added LEDs
Parts:
- J1: symbol Connector:USB_B_Micro -> MC5000_Board-rescue:USB_B_Micro-Connector
Changed lines of the file:
@@
 $Descr A4 11693 8268
 encoding utf-8
-Sheet 2 12
+Sheet 2 13
 Title ""
 Date ""
@@
 $EndDescr
 $Comp
-L Connector:USB_B_Micro J?
+L MC5000_Board-rescue:USB_B_Micro-Connector J?
 U 1 1 602FFA24
 P 3600 3550

Commit message: Cleanup libs
Parts:
- J1: symbol MC5000_Board-rescue:USB_B_Micro-Connector -> LCSC_parts:USB_B_Micro-Connector
Changed lines of the file:
@@
 $EndDescr
 $Comp
-L MC5000_Board-rescue:USB_B_Micro-Connector J?
+L LCSC_parts:USB_B_Micro-Connector J?
 U 1 1 602FFA24
 P 3600 3550
