File: pcb/buzzer.sch (KiCad schematic (older format))
At the start: 8 parts, among them J22 Conn_01x04_Female, J23 Conn_01x04_Female, Q1 S9013

Commit message: Cleanup libs
Parts:
- BZ1: symbol JLC_Parts:MLT-7525 -> LCSC_parts:MLT-7525
- Q1: symbol JLC_Parts:S9013 -> LCSC_parts:S9013
Changed lines of the file:
@@
 $EndDescr
 $Comp
-L JLC_Parts:MLT-7525 BZ1
+L LCSC_parts:MLT-7525 BZ1
 U 1 1 60044231
 P 5950 3500
@@
 $EndComp
 $Comp
-L JLC_Parts:S9013 Q1
+L LCSC_parts:S9013 Q1
 U 1 1 600481C3
 P 5650 4000

Commit message: Added switches
Parts:
- R21: value 100R -> 200R; footprint Resistor_SMD:R_0603_1608Metric -> Resistor_SMD:R_0603_1608Metric_Pad0.98x0.95mm_HandSolder
- R22: value 100k -> 100K; footprint Resistor_SMD:R_0603_1608Metric -> Resistor_SMD:R_0603_1608Metric_Pad0.98x0.95mm_HandSolder
Changed lines of the file:
@@
 $Descr A4 11693 8268
 encoding utf-8
-Sheet 12 13
+Sheet 12 15
 Title ""
 Date ""
@@
 P 4950 4000
 F 0 "R21" V 4743 4000 50  0000 C CNN
-F 1 "100R" V 4834 4000 50  0000 C CNN
-F 2 "Resistor_SMD:R_0603_1608Metric" V 4880 4000 50  0001 C CNN
+F 1 "200R" V 4834 4000 50  0000 C CNN
+F 2 "Resistor_SMD:R_0603_1608Metric_Pad0.98x0.95mm_HandSolder" V 4880 4000 50  0001 C CNN
 F 3 "~" H 4950 4000 50  0001 C CNN
 	1    4950 4000
@@
 P 5300 4250
 F 0 "R22" H 5230 4204 50  0000 R CNN
-F 1 "100k" H 5230 4295 50  0000 R CNN
-F 2 "Resistor_SMD:R_0603_1608Metric" V 5230 4250 50  0001 C CNN
+F 1 "100K" H 5230 4295 50  0000 R CNN
+F 2 "Resistor_SMD:R_0603_1608Metric_Pad0.98x0.95mm_HandSolder" V 5230 4250 50  0001 C CNN
 F 3 "~" H 5300 4250 50  0001 C CNN
 	1    5300 4250
