File: pcb/display.sch (KiCad schematic (older format))
At the start: 10 parts, among them U8 PCA9555PW

Commit message: fixes
Parts:
- added C3, C4: 0.1uF, Capacitor_SMD:C_0603_1608Metric_Pad1.08x0.95mm_HandSolder, symbol Device:C
- added D1: LED, LED_SMD:LED_0805_2012Metric_Pad1.15x1.40mm_HandSolder, symbol Device:LED
- added J14, J15: Conn_01x04_Female, Connector_PinSocket_2.54mm:PinSocket_1x04_P2.54mm_Vertical, symbol Connector:Conn_01x04_Female
- added R10, R11, R12: 10k, Resistor_SMD:R_0603_1608Metric_Pad0.98x0.95mm_HandSolder, symbol Device:R
- added R9: 200R, Resistor_SMD:R_0603_1608Metric_Pad0.98x0.95mm_HandSolder, symbol Device:R
Connections:
- net at U8.1 (~INT): now also J15.3 (Pin_3), R12.1
- net GND: now reaches U8.12 (VSS)
- net GND: now also U8.2 (A1), U8.21 (A0), U8.3 (A2), C3.1, C4.1, D1.1 (K), J15.4 (Pin_4)
- net at U8.16 (IO1_3): now also R9.2
- net at U8.22 (SCL): now also J15.1 (Pin_1), R10.2
- net at U8.23 (SDA): now also J15.2 (Pin_2), R11.1
- net VCC: now reaches U8.24 (VDD)
- net VCC: now also C3.2, C4.2, J14.1 (Pin_1), R10.1, R11.2, R12.2
- new net: D1.2 (A), R9.1
- new net XBUS_Display: J14.3 (Pin_3)
- no-connect marks 0 -> 2
Other:
- moved on the sheet: DS1, R1, R2, R3, R4, R5, R6, R7, R8, U8

Commit message: Added LEDs
Parts:
- U8: symbol Interface_Expansion:PCA9555PW -> MC5000_Board-rescue:PCA9555PW-Interface_Expansion
Changed lines of the file:
@@
 $Descr A4 11693 8268
 encoding utf-8
-Sheet 7 12
+Sheet 7 13
 Title ""
 Date ""
@@
 $EndComp
 $Comp
-L Interface_Expansion:PCA9555PW U8
+L MC5000_Board-rescue:PCA9555PW-Interface_Expansion U8
 U 1 1 6031B3F2
 P 4800 3800
+AR Path="/6031B3F2" Ref="U8"  Part="1"
+AR Path="/60308700/6031B3F2" Ref="U8"  Part="1"
 F 0 "U8" H 4800 2619 50  0000 C CNN
 F 1 "PCA9555PW" H 4800 2710 50  0000 C CNN

Commit message: Cleanup libs
Parts:
- U8: symbol MC5000_Board-rescue:PCA9555PW-Interface_Expansion -> Interface_Expansion:PCA9555PW
Changed lines of the file:
@@
 $EndComp
 $Comp
-L MC5000_Board-rescue:PCA9555PW-Interface_Expansion U8
+L Interface_Expansion:PCA9555PW U8
 U 1 1 6031B3F2
 P 4800 3800

Commit message: Added switches
Parts:
- R10, R11: value 10k -> 2K2
- R12: value 10k -> 100K
Changed lines of the file:
@@
 $Descr A4 11693 8268
 encoding utf-8
-Sheet 7 13
+Sheet 7 15
 Title ""
 Date ""
@@
 P 6250 4900
 F 0 "R10" H 6180 4854 50  0000 R CNN
-F 1 "10k" H 6180 4945 50  0000 R CNN
+F 1 "2K2" H 6180 4945 50  0000 R CNN
 F 2 "Resistor_SMD:R_0603_1608Metric_Pad0.98x0.95mm_HandSolder" V 6180 4900 50  0001 C CNN
 F 3 "~" H 6250 4900 50  0001 C CNN
@@
 P 6450 3900
 F 0 "R12" H 6520 3946 50  0000 L CNN
-F 1 "10k" H 6520 3855 50  0000 L CNN
+F 1 "100K" H 6520 3855 50  0000 L CNN
 F 2 "Resistor_SMD:R_0603_1608Metric_Pad0.98x0.95mm_HandSolder" V 6380 3900 50  0001 C CNN
 F 3 "~" H 6450 3900 50  0001 C CNN
@@
 P 5950 4250
 F 0 "R11" H 5880 4204 50  0000 R CNN
-F 1 "10k" H 5880 4295 50  0000 R CNN
+F 1 "2K2" H 5880 4295 50  0000 R CNN
 F 2 "Resistor_SMD:R_0603_1608Metric_Pad0.98x0.95mm_HandSolder" V 5880 4250 50  0001 C CNN
 F 3 "~" H 5950 4250 50  0001 C CNN
