File: pcb/switches.sch (KiCad schematic (older format))
At the start: 6 parts, among them SW1 SW_MEC_5E

Commit message: Changes
Parts:
- gave numbers to parts that had none: 3
Changed lines of the file:
@@
 $Descr A4 11693 8268
 encoding utf-8
-Sheet 15 15
+Sheet 14 14
 Title ""
 Date ""
@@
 	4200 3700 4300 3700
 $Comp
-L Switch:SW_Push SW?
+L Switch:SW_Push SW2
 U 1 1 6039577E
 P 6300 4550
-AR Path="/6037B4F8/6039577E" Ref="SW?"  Part="1"
+AR Path="/6037B4F8/6039577E" Ref="SW2"  Part="1"
 AR Path="/603926D8/6039577E" Ref="SW?"  Part="1"
-F 0 "SW?" H 6300 4835 50  0000 C CNN
+F 0 "SW2" H 6300 4835 50  0000 C CNN
 F 1 "SW_MEC_5E" H 6300 4744 50  0000 C CNN
 F 2 "Button_Switch_SMD:SW_Push_1P1T_NO_CK_KSC6xxJ" H 6300 4750 50  0001 C CNN
@@
 $EndComp
 $Comp
-L Device:R R?
+L Device:R R35
 U 1 1 60395784
 P 6950 4550
-AR Path="/6037B4F8/60395784" Ref="R?"  Part="1"
+AR Path="/6037B4F8/60395784" Ref="R35"  Part="1"
 AR Path="/603926D8/60395784" Ref="R?"  Part="1"
-F 0 "R?" V 6743 4550 50  0000 C CNN
+F 0 "R35" V 6743 4550 50  0000 C CNN
 F 1 "200R" V 6834 4550 50  0000 C CNN
 F 2 "Resistor_SMD:R_0603_1608Metric_Pad0.98x0.95mm_HandSolder" V 6880 4550 50  0001 C CNN
@@
 $EndComp
 $Comp
-L Device:R R?
+L Device:R R34
 U 1 1 6039578A
 P 6650 4850
-AR Path="/6037B4F8/6039578A" Ref="R?"  Part="1"
+AR Path="/6037B4F8/6039578A" Ref="R34"  Part="1"
 AR Path="/603926D8/6039578A" Ref="R?"  Part="1"
-F 0 "R?" H 6580 4804 50  0000 R CNN
+F 0 "R34" H 6580 4804 50  0000 R CNN
 F 1 "100K" H 6580 4895 50  0000 R CNN
 F 2 "Resistor_SMD:R_0603_1608Metric_Pad0.98x0.95mm_HandSolder" V 6580 4850 50  0001 C CNN
@@
 SWITCH_2
 $Comp
-L power:GND #PWR?
+L power:GND #PWR0118
 U 1 1 60395796
 P 6650 5150
-AR Path="/6037B4F8/60395796" Ref="#PWR?"  Part="1"
+AR Path="/6037B4F8/60395796" Ref="#PWR0118"  Part="1"
 AR Path="/603926D8/60395796" Ref="#PWR?"  Part="1"
-F 0 "#PWR?" H 6650 4900 50  0001 C CNN
+F 0 "#PWR0118" H 6650 4900 50  0001 C CNN
 F 1 "GND" H 6655 4977 50  0000 C CNN
 F 2 "" H 6650 5150 50  0001 C CNN
@@
 	6650 5150 6650 5000
 $Comp
-L power:VCC #PWR?
+L power:VCC #PWR0120
 U 1 1 6039579D
 P 6000 4550
-AR Path="/6037B4F8/6039579D" Ref="#PWR?"  Part="1"
+AR Path="/6037B4F8/6039579D" Ref="#PWR0120"  Part="1"
 AR Path="/603926D8/6039579D" Ref="#PWR?"  Part="1"
-F 0 "#PWR?" H 6000 4400 50  0001 C CNN
+F 0 "#PWR0120" H 6000 4400 50  0001 C CNN
 F 1 "VCC" V 6015 4677 50  0000 L CNN
 F 2 "" H 6000 4550 50  0001 C CNN
