File: pcb/connection_block.sch (KiCad schematic (older format))
At the start: 2 parts, among them J24 Conn_01x04_Female, J25 Conn_01x05_Female

Commit message: XBus changes; PCB changes
Parts:
- J24: LCSC (none) -> C124413
- J25: LCSC (none) -> C718240
Changed lines of the file:
@@
 F 2 "Connector_PinSocket_2.54mm:PinSocket_1x04_P2.54mm_Vertical" H 5800 3550 50  0001 C CNN
 F 3 "~" H 5800 3550 50  0001 C CNN
+F 4 "C124413" H 5800 3550 50  0001 C CNN "LCSC"
 	1    5800 3550
 	1    0    0    -1
@@
 F 2 "Connector_PinSocket_2.54mm:PinSocket_1x05_P2.54mm_Vertical" H 5800 2900 50  0001 C CNN
 F 3 "~" H 5800 2900 50  0001 C CNN
+F 4 "C718240" H 5800 2900 50  0001 C CNN "LCSC"
 	1    5800 2900
 	1    0    0    -1

Commit message: Production board
Parts:
- J24: footprint Connector_PinSocket_2.54mm:PinSocket_1x04_P2.54mm_Vertical -> LCSC_parts:PinSocket_1x04_P2.54mm_Vertical_centered
- J25: footprint Connector_PinSocket_2.54mm:PinSocket_1x05_P2.54mm_Vertical -> LCSC_parts:PinSocket_1x05_P2.54mm_Vertical_centered
Changed lines of the file:
@@
 $Descr A4 11693 8268
 encoding utf-8
-Sheet 17 17
+Sheet 17 11
 Title ""
 Date ""
@@
 F 0 "J24" H 5828 3526 50  0000 L CNN
 F 1 "Conn_01x04_Female" H 5828 3435 50  0000 L CNN
-F 2 "Connector_PinSocket_2.54mm:PinSocket_1x04_P2.54mm_Vertical" H 5800 3550 50  0001 C CNN
+F 2 "LCSC_parts:PinSocket_1x04_P2.54mm_Vertical_centered" H 5800 3550 50  0001 C CNN
 F 3 "~" H 5800 3550 50  0001 C CNN
 F 4 "C124413" H 5800 3550 50  0001 C CNN "LCSC"
@@
 F 0 "J25" H 5828 2926 50  0000 L CNN
 F 1 "Conn_01x05_Female" H 5828 2835 50  0000 L CNN
-F 2 "Connector_PinSocket_2.54mm:PinSocket_1x05_P2.54mm_Vertical" H 5800 2900 50  0001 C CNN
+F 2 "LCSC_parts:PinSocket_1x05_P2.54mm_Vertical_centered" H 5800 2900 50  0001 C CNN
 F 3 "~" H 5800 2900 50  0001 C CNN
 F 4 "C718240" H 5800 2900 50  0001 C CNN "LCSC"
